File: boards/mejoras/G/G.sch (EAGLE design)
At the start: 34 parts, among them J1 XT60-M, J2 XT60-M, J3 XT60-M, J4 XT60-M, J5 XT60-M, J6 XT60-M, Q1 IRFR7440PBF, Q2 IRFR7440PBF

Commit message: changes to g circuit
Parts:
- L1: value MSS7341 -> DR125; device inductor-coilcraft:MSS7341 -> inductors:DR125
Changed lines of the file:
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@@
 <?xml version="1.0" encoding="utf-8"?>
 <!DOCTYPE eagle SYSTEM "eagle.dtd">
-<eagle version="9.6.2">
+<eagle version="9.6.0">
 <drawing>
 <settings>
@@
 <part name="R13" library="rcl" library_urn="urn:adsk.eagle:library:334" deviceset="R-US_" device="M1206" package3d_urn="urn:adsk.eagle:package:23566/2"/>
 <part name="IC3" library="linear" library_urn="urn:adsk.eagle:library:262" deviceset="LM2596S" device="" package3d_urn="urn:adsk.eagle:package:16438/2"/>
-<part name="L1" library="inductor-coilcraft" library_urn="urn:adsk.eagle:library:240" deviceset="MSS7341" device="" package3d_urn="urn:adsk.eagle:package:14501/1"/>
 <part name="D2" library="diode" library_urn="urn:adsk.eagle:library:210" deviceset="MBRS3*0T3" device="" package3d_urn="urn:adsk.eagle:package:43425/2" technology="2"/>
 <part name="R14" library="rcl" library_urn="urn:adsk.eagle:library:334" deviceset="R-US_" device="M1206" package3d_urn="urn:adsk.eagle:package:23566/2"/>
@@
 <part name="C5" library="adafruit" library_urn="urn:adsk.eagle:library:420" deviceset="CPOL-US" device="153CLV-1014" package3d_urn="urn:adsk.eagle:package:6240463/1"/>
 <part name="C1" library="adafruit" library_urn="urn:adsk.eagle:library:420" deviceset="CPOL-US" device="153CLV-1014" package3d_urn="urn:adsk.eagle:package:6240463/1"/>
+<part name="L1" library="inductors" library_urn="urn:adsk.eagle:library:243" deviceset="DR125" device="" package3d_urn="urn:adsk.eagle:package:15121/1"/>
 </parts>
 <sheets>
@@
 <attribute name="VALUE" x="-78.74" y="138.43" size="1.778" layer="96"/>
 </instance>
-<instance part="L1" gate="G$1" x="-43.18" y="134.62" smashed="yes">
-<attribute name="NAME" x="-46.99" y="136.1186" size="1.778" layer="95"/>
-<attribute name="VALUE" x="-46.99" y="131.318" size="1.778" layer="96"/>
-</instance>
 <instance part="D2" gate="G$1" x="-53.34" y="127" smashed="yes" rot="R90">
 <attribute name="NAME" x="-55.245" y="124.714" size="1.778" layer="95" rot="R90"/>
@@
 <attribute name="NAME" x="-24.384" y="94.615" size="1.778" layer="95"/>
 <attribute name="VALUE" x="-24.384" y="89.789" size="1.778" layer="96"/>
+</instance>
+<instance part="L1" gate="G$1" x="-45.72" y="139.7" smashed="yes">
+<attribute name="NAME" x="-49.53" y="141.986" size="1.778" layer="95"/>
+<attribute name="VALUE" x="-49.657" y="136.652" size="1.778" layer="96"/>
 </instance>
 </instances>
@@
 </segment>
 <segment>
-<wire x1="-38.1" y1="134.62" x2="-35.56" y2="134.62" width="0.1524" layer="91"/>
 <wire x1="-35.56" y1="134.62" x2="-35.56" y2="127" width="0.1524" layer="91"/>
-<pinref part="L1" gate="G$1" pin="2"/>
 <pinref part="IC3" gate="G$1" pin="FB"/>
 <wire x1="-71.12" y1="129.54" x2="-63.5" y2="129.54" width="0.1524" layer="91"/>
@@
 <label x="-27.94" y="134.62" size="1.778" layer="95"/>
 <pinref part="C4" gate="G$1" pin="+"/>
+<pinref part="L1" gate="G$1" pin="2"/>
+<wire x1="-38.1" y1="139.7" x2="-38.1" y2="134.62" width="0.1524" layer="91"/>
+<wire x1="-38.1" y1="134.62" x2="-35.56" y2="134.62" width="0.1524" layer="91"/>
 </segment>
 </net>
@@
 <segment>
 <pinref part="IC3" gate="G$1" pin="OUT"/>
-<wire x1="-71.12" y1="134.62" x2="-53.34" y2="134.62" width="0.1524" layer="91"/>
+<wire x1="-71.12" y1="134.62" x2="-58.42" y2="134.62" width="0.1524" layer="91"/>
+<wire x1="-58.42" y1="134.62" x2="-53.34" y2="134.62" width="0.1524" layer="91"/>
 <wire x1="-53.34" y1="134.62" x2="-53.34" y2="129.54" width="0.1524" layer="91"/>
-<wire x1="-53.34" y1="134.62" x2="-48.26" y2="134.62" width="0.1524" layer="91"/>
-<junction x="-53.34" y="134.62"/>
+<pinref part="D2" gate="G$1" pin="C"/>
 <pinref part="L1" gate="G$1" pin="1"/>
-<pinref part="D2" gate="G$1" pin="C"/>
-</segment>
-</net>
+<wire x1="-53.34" y1="139.7" x2="-58.42" y2="139.7" width="0.1524" layer="91"/>
+<wire x1="-58.42" y1="139.7" x2="-58.42" y2="134.62" width="0.1524" layer="91"/>
+<junction x="-58.42" y="134.62"/>
+</segment>
+</net>

Commit message: corrected bug
Connections:
- removed net POWER: U$2.VBAT_12
- net VPOWER: now also U$2.VBAT_12
Changed lines of the file:
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@@
 <?xml version="1.0" encoding="utf-8"?>
 <!DOCTYPE eagle SYSTEM "eagle.dtd">
-<eagle version="9.6.0">
+<eagle version="9.6.2">
 <drawing>
 <settings>
@@
 <pinref part="C1" gate="G$1" pin="+"/>
 </segment>
+<segment>
+<pinref part="U$2" gate="G$1" pin="VBAT_12"/>
+<wire x1="373.38" y1="127" x2="388.62" y2="127" width="0.1524" layer="91"/>
+<label x="381" y="127" size="1.778" layer="95"/>
+</segment>
 </net>
 <net name="5V" class="0">
@@
 </segment>
 </net>
-<net name="POWER" class="0">
-<segment>
-<pinref part="U$2" gate="G$1" pin="VBAT_12"/>
-<wire x1="373.38" y1="127" x2="388.62" y2="127" width="0.1524" layer="91"/>
-<label x="383.54" y="127" size="1.778" layer="95"/>
-</segment>
-</net>

Commit message: udpated new circuits
Parts:
- added R1, R16: (no value), rcl:R-US_M1206
Connections:
- new net N$19: R1.1, U$1.CS_8
- new net N$20: R16.1, U$2.CS_8
- net GND: now also R1.2, R16.2
Changed lines of the file:
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@@
 <part name="C1" library="adafruit" library_urn="urn:adsk.eagle:library:420" deviceset="CPOL-US" device="153CLV-1014" package3d_urn="urn:adsk.eagle:package:6240463/1"/>
 <part name="L1" library="inductors" library_urn="urn:adsk.eagle:library:243" deviceset="DR125" device="" package3d_urn="urn:adsk.eagle:package:15121/1"/>
+<part name="R1" library="rcl" library_urn="urn:adsk.eagle:library:334" deviceset="R-US_" device="M1206" package3d_urn="urn:adsk.eagle:package:23566/2"/>
+<part name="R16" library="rcl" library_urn="urn:adsk.eagle:library:334" deviceset="R-US_" device="M1206" package3d_urn="urn:adsk.eagle:package:23566/2"/>
 </parts>
 <sheets>
@@
 <attribute name="NAME" x="-49.53" y="141.986" size="1.778" layer="95"/>
 <attribute name="VALUE" x="-49.657" y="136.652" size="1.778" layer="96"/>
+</instance>
+<instance part="R1" gate="G$1" x="132.08" y="91.44" smashed="yes" rot="R180">
+<attribute name="NAME" x="135.89" y="89.9414" size="1.778" layer="95" rot="R180"/>
+<attribute name="VALUE" x="135.89" y="94.742" size="1.778" layer="96" rot="R180"/>
+</instance>
+<instance part="R16" gate="G$1" x="279.4" y="88.9" smashed="yes" rot="R180">
+<attribute name="NAME" x="283.21" y="87.4014" size="1.778" layer="95" rot="R180"/>
+<attribute name="VALUE" x="283.21" y="92.202" size="1.778" layer="96" rot="R180"/>
 </instance>
 </instances>
@@
 <pinref part="C1" gate="G$1" pin="-"/>
 </segment>
+<segment>
+<pinref part="R1" gate="G$1" pin="2"/>
+<wire x1="127" y1="91.44" x2="119.38" y2="91.44" width="0.1524" layer="91"/>
+<label x="119.38" y="91.44" size="1.778" layer="95"/>
+</segment>
+<segment>
+<pinref part="R16" gate="G$1" pin="2"/>
+<wire x1="274.32" y1="88.9" x2="266.7" y2="88.9" width="0.1524" layer="91"/>
+<label x="266.7" y="91.44" size="1.778" layer="95"/>
+</segment>
 </net>
 <net name="VPOWER" class="0">
@@
 <segment>
 <pinref part="U$1" gate="G$1" pin="ENB/DIAGB_9"/>
-<wire x1="160.02" y1="109.22" x2="157.48" y2="109.22" width="0.1524" layer="91"/>
-<wire x1="157.48" y1="109.22" x2="157.48" y2="114.3" width="0.1524" layer="91"/>
+<wire x1="160.02" y1="109.22" x2="154.94" y2="109.22" width="0.1524" layer="91"/>
+<wire x1="154.94" y1="109.22" x2="154.94" y2="114.3" width="0.1524" layer="91"/>
 <pinref part="R8" gate="G$1" pin="1"/>
-<wire x1="157.48" y1="114.3" x2="154.94" y2="114.3" width="0.1524" layer="91"/>
 </segment>
 </net>
@@
 </segment>
 </net>
+<net name="N$19" class="0">
+<segment>
+<pinref part="R1" gate="G$1" pin="1"/>
+<wire x1="137.16" y1="91.44" x2="144.78" y2="91.44" width="0.1524" layer="91"/>
+<wire x1="144.78" y1="91.44" x2="144.78" y2="99.06" width="0.1524" layer="91"/>
+<wire x1="144.78" y1="99.06" x2="157.48" y2="99.06" width="0.1524" layer="91"/>
+<wire x1="157.48" y1="99.06" x2="157.48" y2="114.3" width="0.1524" layer="91"/>
+<pinref part="U$1" gate="G$1" pin="CS_8"/>
+<wire x1="157.48" y1="114.3" x2="160.02" y2="114.3" width="0.1524" layer="91"/>
+</segment>
+</net>
+<net name="N$20" class="0">
+<segment>
+<pinref part="R16" gate="G$1" pin="1"/>
+<wire x1="284.48" y1="88.9" x2="309.88" y2="88.9" width="0.1524" layer="91"/>
+<wire x1="309.88" y1="88.9" x2="309.88" y2="109.22" width="0.1524" layer="91"/>
+<pinref part="U$2" gate="G$1" pin="CS_8"/>
+<wire x1="309.88" y1="109.22" x2="312.42" y2="109.22" width="0.1524" layer="91"/>
+</segment>
+</net>
