File: boards/mejoras/H/H.brd (EAGLE design)
At the start: 100 x 35 mm, 37 parts, among them IC1 PIC18F4455_TQFP

Commit message: updated boards
Connections:
- net 5V: now also R4.1, R5.1, R6.1, R7.1
- net GND: no longer R4.1, R5.1, R6.1, R7.1
Routing:
- net GND: track 391.0 -> 367.0 mm
- net 5V: track 251.5 -> 269.8 mm
- net PWM1: track 53.2 -> 51.2 mm
- net B2: track 39.8 -> 38.7 mm
- net B1: track 40.5 -> 39.4 mm
- net CNY3: track 83.4 -> 84.1 mm
- net PWM2: track 20.6 -> 21.2 mm
